File: Diagnostic_Panel/Diagnostic_Panel.kicad_pcb (KiCad board)
At the start: 2 copper layers, 81.7 x 103 mm, 17 parts, among them P1 CONN_2

Commit message: Added revision text
Other:
- board text added: "CySat Diagnostic Panel: Rev B 4/15/2015"
