File: Top_Panel/Top_Panel.kicad_pcb (KiCad board)
At the start: 2 copper layers, 99 x 99 mm, 26 parts, among them P1 CONN_2, P2 CONN_1, P3 CONN_1, P4 CONN_1, P5 CONN_1, P6 CONN_1, P7 CONN_1, P8 CONN_1

Commit message: Added revision text
Other:
- board text added: "CySat Top Panel: Rev C 4/15/2015"
