File: SolarTestBoard/SolarPanelTest.kicad_pcb (KiCad board)
At the start: 2 copper layers, 176.7 x 115.8 mm, 14 parts, among them J1 Conn_01x04, J2 Conn_01x10

Commit message: Changed footprints to add troubleshooting jumpers and the molex connector
Parts:
- added J3: Split Cells, Pin_Headers:Pin_Header_Straight_1x02_Pitch2.54mm, F.Cu at (242.6, 111.8)
- added J4: Two Cells, Pin_Headers:Pin_Header_Straight_1x02_Pitch2.54mm, F.Cu at (227.3, 127.0)
- J1: footprint Pin_Headers:Pin_Header_Straight_1x04_Pitch2.54mm -> Connectors_Molex:Molex_PicoBlade_53398-0471_04x1.25mm_Straight
- J2: value Conn_01x10 -> Two Cells; footprint Pin_Headers:Pin_Header_Straight_1x10_Pitch2.54mm -> Pin_Headers:Pin_Header_Straight_1x02_Pitch2.54mm
- moved J2 64.9 mm to (242.6, 104.1), turned to 270 degrees
- moved J1 5.24 mm to (104.1, 96.5), turned to 270 degrees
Connections:
- J1 pad 1: G -> F
- J1 pad 2: C -> F
- J1 pad 3: B -> A
- J2 pad 1: A -> B
- J2 pad 2: B -> A
- SC1 pad 2: B -> F
- SC10 pad 2: G -> F
- SC11 pad 2: G -> F
- SC12 pad 1: Net-(SC12-Pad1) -> D
- SC12 pad 2: G -> E
- SC2 pad 1: C -> A
- SC3 pad 1: C -> A
- SC4 pad 2: B -> F
- SC5 pad 1: C -> A
- SC6 pad 1: C -> A
- SC7 pad 1: C -> B
- SC7 pad 2: Net-(SC12-Pad1) -> C
- SC8 pad 2: G -> F
- SC9 pad 2: G -> F
Routing:
- net F: track 0.00 -> 500.9 mm, vias 0 -> 2
- net B: track 389.5 -> 18.0 mm, vias 1 -> 0
- net C: track 253.0 -> 5.46 mm, vias 2 -> 0
- net G: track 200.4 -> 0.00 mm
- net A: track 310.6 -> 386.2 mm, vias 1 -> 2
- net D: track 0.00 -> 24.1 mm
- net E: track 0.00 -> 21.8 mm
- net Net-(SC12-Pad1): track 16.0 -> 0.00 mm
Other:
- board text removed: "VCC"
- board text removed: "VSS"

Commit message: Finished v1
Parts:
- added G***: LOGO, photo:safetySat, B.Cu at (189.2, 63.5)
- added LOGO: , motherboard:LOGO, F.Cu at (105.4, 123.2)
Routing:
- net A: track 386.2 -> 493.0 mm
- net F: track 500.9 -> 607.4 mm
- net Net-(SC2-Pad2): track 16.0 -> 29.4 mm
- net Net-(SC3-Pad2): track 16.0 -> 29.4 mm
- net Net-(SC10-Pad1): track 27.2 -> 40.6 mm
- net Net-(SC11-Pad1): track 21.6 -> 24.8 mm
- net D: track 24.1 -> 27.2 mm
- net B: track 18.0 -> 21.1 mm
Other:
- net class Default: clearance 0.2 -> 0.2032
- rule trace_clearance: 0.2 -> 0.2032
