File: schematic/AntennaDeployBracket/AntennaDeploymentBracket.kicad_pcb (KiCad board)
At the start: 2 copper layers, 18.9 x 17.3 mm, 6 parts, among them J1 Conn_01x02

Commit message: Finished Right, Back 90% done.
Parts:
- moved R1 2.53 mm to (125.4, 97.8)
- moved J1 2.41 mm to (125.1, 103.0)
Other:
- outline, holes or cut-outs redrawn
Changed lines of the file:
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@@
     (thickness 1.6)
     (drawings 13)
-    (tracks 4)
+    (tracks 5)
     (zones 0)
     (modules 6)
@@
   )
   (module Wire_Pads:SolderWirePad_2x_1mmDrill (layer F.Cu)
-    (at 125.095 100.584)
+    (at 125.095 102.997)
     (fp_text reference J1 (at 0 -3.81) (layer F.SilkS)
       (effects (font (size 1 1) (thickness 0.15)))
@@
   )
   (module AntennaDeploymentBracket:AntennaDeploymentBracket (layer F.Cu)
-    (at 125.3845 95.2246)
+    (at 125.3744 97.7519)
     (fp_text reference R1 (at -4.3535 1.8034) (layer F.SilkS)
       (effects (font (size 1 1) (thickness 0.15)))
@@
     (pad 1 thru_hole circle (at 0 0) (size 3.5 3.5) (drill 3) (layers *.Cu *.Mask))
   )
-  (gr_text "Antenna\nDeployment\nBoard" (at 125.222 104.013) (layer F.SilkS)
+  (gr_text "Antenna\nDeployment\nBoard" (at 125.222 93.218) (layer F.SilkS)
     (effects (font (size 0.8 0.8) (thickness 0.2)))
   )
@@
     (effects (font (size 1.5 1.5) (thickness 0.3)))
   )
-  (gr_text "Burn, baby, burn!" (at 125.222 98.679) (layer F.SilkS)
+  (gr_text "Burn, baby, burn!" (at 125.095 100.838) (layer F.SilkS)
     (effects (font (size 1.5 1.42) (thickness 0.3)))
   )
@@
   (gr_line (start 115.697 106.172) (end 134.62 106.172) (layer Edge.Cuts) (width 0.15))
   (gr_line (start 115.697 88.9) (end 115.697 106.172) (layer Edge.Cuts) (width 0.15))
-  (gr_arc (start 123.19 95.25) (end 123.19 93.726) (angle -180) (layer Edge.Cuts) (width 0.15))
-  (gr_arc (start 127.127 95.25) (end 127.127 96.774) (angle -180) (layer Edge.Cuts) (width 0.15))
-  (gr_line (start 123.19 97.536) (end 123.19 92.71) (layer Edge.Cuts) (width 0.15))
-  (gr_line (start 127.127 97.536) (end 123.19 97.536) (layer Edge.Cuts) (width 0.15))
-  (gr_line (start 127.127 92.71) (end 127.127 97.536) (layer Edge.Cuts) (width 0.15))
-  (gr_line (start 123.19 92.71) (end 127.127 92.71) (layer Edge.Cuts) (width 0.15))
-  (segment (start 120.622 98.016) (end 120.622 95.25) (width 0.25) (layer F.Cu) (net 1))
-  (segment (start 123.19 100.584) (end 120.622 98.016) (width 0.25) (layer F.Cu) (net 1))
-  (segment (start 129.8041 97.7799) (end 127 100.584) (width 0.25) (layer F.Cu) (net 2))
-  (segment (start 129.8041 95.2627) (end 129.8041 97.7799) (width 0.25) (layer F.Cu) (net 2))
+  (gr_arc (start 123.19 97.663) (end 123.19 96.139) (angle -180) (layer Edge.Cuts) (width 0.15))
+  (gr_arc (start 127.127 97.663) (end 127.127 99.187) (angle -180) (layer Edge.Cuts) (width 0.15))
+  (gr_line (start 123.19 99.949) (end 123.19 95.123) (layer Edge.Cuts) (width 0.15))
+  (gr_line (start 127.127 99.949) (end 123.19 99.949) (layer Edge.Cuts) (width 0.15))
+  (gr_line (start 127.127 95.123) (end 127.127 99.949) (layer Edge.Cuts) (width 0.15))
+  (gr_line (start 123.19 95.123) (end 127.127 95.123) (layer Edge.Cuts) (width 0.15))
+  (segment (start 120.622 100.429) (end 120.622 97.663) (width 0.25) (layer F.Cu) (net 1))
+  (segment (start 123.19 102.997) (end 120.622 100.429) (width 0.25) (layer F.Cu) (net 1))
+  (segment (start 129.8041 100.1929) (end 127 102.997) (width 0.25) (layer F.Cu) (net 2))
+  (segment (start 129.794 100.1828) (end 129.794 97.79) (width 0.25) (layer F.Cu) (net 2))
+  (segment (start 129.8041 100.1929) (end 129.794 100.1828) (width 0.25) (layer F.Cu) (net 2))
 )
