File: schematic/Sidepanels/RightSidePanel/RightSidePanel.kicad_pcb (KiCad board)
At the start: 2 copper layers, 327.5 x 83 mm, 7 parts, among them J1 Conn_01x04

Commit message: FINALLY got the pcb art I wanted
Parts:
- removed G***: LOGO, SolarPanelFoot:CySat1
- added ?: , CysatSide:CySatLogo, F.Cu at (156.6, 131.9)
