File: schematic/Sidepanels_2019/X+/X+.kicad_pcb (KiCad board)
At the start: 2 copper layers, 327.5 x 83 mm, 33 parts, among them J1 Conn_01x04, J2 Conn_01x02

Commit message: Flipped and added TrisolX cells
Parts:
- added D16: D_Schottky, CySat footprints:Toshiba_CUS08F30, B.Cu at (268.5, -67.5)
- added SC17: Solar_Cell, CySat footprints:TriSelectSolarPanel_Left_Handed, F.Cu at (299.9, -60.0)
- SC10, SC11, SC12, SC13, SC14, SC15, SC16, SC5, SC6, SC7, SC8, SC9: footprint CySat footprints:TriSelectSolarPanel -> CySat footprints:TriSelectSolarPanel_Left_Handed
- moved SC13 13.0 mm to (90.4, -56.0)
- moved SC7 12.5 mm to (106.8, -50.2)
- moved SC9 12.5 mm to (106.8, -41.6)
- moved SC10 12.5 mm to (106.8, -75.9)
- moved SC11 12.5 mm to (106.8, -67.3)
- moved SC12 12.5 mm to (106.8, -58.7)
- moved SC5 12.5 mm to (106.8, -101.6)
- moved SC6 12.5 mm to (106.8, -93.0)
- moved SC8 12.5 mm to (106.8, -84.5)
- moved SC15 12.0 mm to (-1.96, -55.6)
- moved SC16 11.3 mm to (299.8, -100.1)
- moved SC14 7.31 mm to (81.9, -93.0)
Routing:
- net VCC: track 42.7 -> 78.8 mm, vias 16 -> 17
- net VSS: track 379.6 -> 409.0 mm, vias 28 -> 29

Commit message: Flipped/removed Trisol Cells
Parts:
- removed D16: D_Schottky, CySat footprints:Toshiba_CUS08F30
- removed SC17: Solar_Cell, CySat footprints:TriSelectSolarPanel_Left_Handed
- SC10, SC11, SC12, SC13, SC14, SC15, SC16, SC7, SC8, SC9: footprint CySat footprints:TriSelectSolarPanel_Left_Handed -> CySat footprints:TriSelectSolarPanel
- moved SC14 52.4 mm to (95.9, -42.5), turned to 0 degrees
- moved SC6 43.4 mm to (90.8, -52.7), turned to 90 degrees
- moved SC12 21.1 mm to (95.8, -76.7)
- moved SC10 21.1 mm to (95.8, -93.9)
- moved SC11 21.1 mm to (95.8, -85.3)
- moved SC7 21.1 mm to (95.8, -68.2)
- moved SC8 21.1 mm to (95.8, -102.4)
- moved SC9 21.1 mm to (95.8, -59.6)
- moved SC5 18.0 mm to (90.7, -93.5), turned to 90 degrees
- moved SC16 11.0 mm to (299.8, -111.1)
- moved SC13 7.35 mm to (95.9, -51.0), turned to 0 degrees
- moved SC15 4.71 mm to (-2.45, -60.3)
Routing:
- net VSS: track 409.0 -> 395.7 mm, vias 29 -> 28
- net VCC: track 78.8 -> 79.8 mm, vias 17 -> 16

Commit message: Update to X panels
Routing completed on both, solar panel change out complete on X+.  Re-did library and page settings.  DRC checks out.
Parts:
- removed D10, D11, D12, D13, D14, D2, D3, D4, D5, D6, D7, D8, D9: D_Schottky, CySat footprints:Toshiba_CUS08F30
- removed D15: D_Photo, CySat footprints:Sun_Sensor
- removed SC10, SC11, SC12, SC13, SC14, SC15, SC16, SC8, SC9: Solar_Cell, CySat footprints:TriSelectSolarPanel
- D1: value D_Schottky -> D_Photo; footprint CySat footprints:Toshiba_CUS08F30 -> Diode_SMD:D_0805_2012Metric; moved to F.Cu
- SC1, SC2: footprint CySat footprints:ISS_SolarCell -> CySat_Solar:Spectrolab
- SC3, SC4: footprint CySat footprints:Spectrolab -> CySat_Solar:Spectrolab
- SC5, SC6: footprint CySat footprints:TriSelectSolarPanel_Left_Handed -> CySat_Solar:Spectrolab
- SC7: footprint CySat footprints:TriSelectSolarPanel -> CySat_Solar:Spectrolab
- moved SC1 463.8 mm to (417.8, 166.4), turned to 270 degrees
- moved SC2 321.4 mm to (373.4, 168.9), turned to 270 degrees
- moved D1 305.0 mm to (375.5, 207.3), turned to 0 degrees
- moved SC5 301.9 mm to (240.0, 168.9), turned to 270 degrees
- moved J2 288.6 mm to (427.4, 174.1)
- moved J1 288.6 mm to (427.4, 163.0)
- moved SC3 272.5 mm to (328.9, 168.9)
- moved SC4 245.9 mm to (284.5, 168.9)
- moved SC6 245.1 mm to (195.6, 168.9), turned to 270 degrees
- moved SC7 243.4 mm to (151.1, 168.9), turned to 270 degrees
Connections:
- D1 pad 1: VCC -> Net-(D1-Pad1)
- D1 pad 2: VSS -> Net-(D1-Pad2)
- J2 pad 1: Net-(D15-Pad2) -> Net-(D1-Pad2)
- J2 pad 2: Net-(D15-Pad1) -> Net-(D1-Pad1)
Routing:
- net VSS: track 395.7 -> 52.2 mm, vias 28 -> 7
- net Net-(D1-Pad1): track 0.00 -> 70.8 mm, vias 0 -> 1
- net Net-(D15-Pad2): track 68.6 -> 0.00 mm, vias 1 -> 0
- net Net-(D1-Pad2): track 0.00 -> 68.4 mm, vias 0 -> 1
- net Net-(D15-Pad1): track 64.9 -> 0.00 mm, vias 1 -> 0
- net VCC: track 79.8 -> 26.5 mm, vias 16 -> 1
Other:
- outline, holes or cut-outs redrawn
- board text removed: "X+"

Commit message: Update to all boards
Added labels to boards to resolve issue #2
Added names of students and faculty to boards
Generated Step files to resolve issue #4, please note the export does include the silkscreen.
Other:
- board text added: "CySat-1 2014-2020 Student Roster Trent Allison, Logan Anderson, Manikrishnakumar Bhuma, Conner Born, Brian Bradford*, Benjamin Briggs, William Brown*, Kyle Caponi*, Ola Carnahan, Brian Caskey, Ricardo Cosme-Bell, Jared Danner, Jacob Drahos*, Leo Freier, Bryan Friestad*, Joshua Gilmore*, Jacob Goldenberg*, Angel Gonzalez, Ian Gonzalez-Alfonzo, Luke Gordon*, Benjamin Halley*, Ryan Hansen, Samuel Ha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"
- board text added: "CySat-1 X+ Panel"
- board text added: "Faculty Advisors Matthew E. Nelson Tomas Gonzalez-Torres Dae Young Lee Phillip Jones Special Thanks To: Iowa Space Grant Consortium Aerospace Enigneering Department ISU Foundation"
Changed lines of the file:
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@@
   (general
     (thickness 1.6)
-    (drawings 122)
+    (drawings 125)
     (tracks 60)
     (zones 0)
@@
   )
   (layers
-    (0 F.Cu signal)
-    (31 B.Cu signal)
+    (0 F.Cu signal hide)
+    (31 B.Cu signal hide)
     (32 B.Adhes user)
     (33 F.Adhes user)
@@
       (rotate (xyz 180 0 0))
     )
+  )
+  (gr_text "CySat-1 X+ Panel" (at 167.64 130.81) (layer F.SilkS)
+    (effects (font (size 1.5 1.5) (thickness 0.3)))
+  )
+  (gr_text "Faculty Advisors\n\nMatthew E. Nelson\nTomas Gonzalez-Torres\nDae Young Lee\nPhillip Jones\n\nSpecial Thanks To:\nIowa Space Grant Consortium\nAerospace Enigneering Department\nISU Foundation" (at 296.545 168.275 270) (layer B.SilkS)
+    (effects (font (size 1.5 1.5) (thickness 0.3)) (justify mirror))
+  )
+  (gr_text "CySat-1 2014-2020 Student Roster\n\nTrent Allison, Logan Anderson, Manikrishnakumar Bhuma, \nConner Born, Brian Bradford*, Benjamin Briggs, William Brown*, \nKyle Caponi*, Ola Carnahan, Brian Caskey, Ricardo Cosme-Bell, \nJared Danner, Jacob Drahos*, Leo Freier, Bryan Friestad*, \nJoshua Gilmore*, Jacob Goldenberg*, Angel Gonzalez, \nIan Gonzalez-Alfonzo, Luke Gordon*, Benjamin Halley*, \nRyan Hansen, Samuel Hartman, Shane Hickson*, Nolan Jessen*, \nDerek Johnson, Yusuke Katagiri, Brian Kempa*, Mackenzie Kilcoin*, \nMaxwell Kiley, Travis King*, Chase Kirchner, Alfin Koshy, \nArunmoli Krishnan, Kate Larsson, Yiqi Liang, Gage Lochner, \nGrant Mathiason, Bryce Miles, Collin Monsees, Kyle Muehlenthaler, \nMatthew Paavola*, Peter Papadopolous*, Ryan Peterson, \nJeff Philogene, Matthew Plewa, Sierra Quenzer, Vaicunth Rajan, \nJordan Reese, Benjamin Reichert, William Rickert*, Samuel Ruhlin*, \nMichael Schoenke, William Searight, Rami Shoukih*, Samuel Sie, \nTalon Stromgren, Benjamin Sweet*, Kelly Thompson, Kyle Uhlenhake*, \nRoss Wagner, Nate Wernimont*, James Wigda, Xiangzhu Yan\n\n* Denotes student in a leadership role\n" (at 360.045 168.275 270) (layer B.SilkS)
+    (effects (font (size 1.5 1.5) (thickness 0.3)) (justify mirror))
   )
   (gr_arc (start 143.4766 145.034) (end 143.4846 147.7264) (angle -89.28409539) (layer Edge.Cuts) (width 0.15))
@@
   (segment (start 426.12 173.355) (end 426.2 173.435) (width 0.25) (layer B.Cu) (net 4))
   (segment (start 402.59 173.355) (end 426.12 173.355) (width 0.25) (layer B.Cu) (net 4))
-  (zone (net 2) (net_name VCC) (layer F.Cu) (hatch edge 0.508)
-    (connect_pads (clearance 0.508))
-    (min_thickness 0.254)
-    (fill yes (arc_segments 32) (thermal_gap 0.508) (thermal_bridge_width 0.508))
-    (polygon
-      (pts
-        (xy 314.9092 -34.3662) (xy 314.8838 -117.348) (xy -6.2484 -117.348) (xy -6.223 -100.0252) (xy -6.3754 -99.2124)
-        (xy -6.6548 -98.6028) (xy -7.1374 -98.0948) (xy -7.6708 -97.7138) (xy -8.2804 -97.4598) (xy -9.1694 -97.3836)
-        (xy -12.5984 -97.409) (xy -12.5984 -34.3662)
-      )
-    )
-  )
   (zone (net 1) (net_name VSS) (layer B.Cu) (hatch edge 0.508)
     (connect_pads (clearance 0.508))

Commit message: updated on save
Parts:
- moved SC1 2.28 mm to (417.8, 168.7)
Routing:
- net VSS: track 52.2 -> 53.0 mm
Other:
- outline, holes or cut-outs redrawn
- rule pad_to_mask_clearance: 0.051 -> 0

Commit message: Push of all changes made for June update
Major change was in the solar cell and creating a new library based on the old one.
Parts:
- SC1, SC2, SC3, SC4, SC5, SC6, SC7: footprint CySat_Solar:Spectrolab -> CySat:Spectrolabs_UTJ
- moved D1 41.3 mm to (416.6, 203.2), turned to 180 degrees
- moved SC3 24.2 mm to (353.1, 170.2)
- moved SC2 22.9 mm to (396.2, 170.2)
- moved SC4 22.9 mm to (307.3, 170.2)
- moved SC1 21.7 mm to (439.4, 170.2)
- moved SC5 21.6 mm to (261.6, 170.2)
- moved SC6 20.3 mm to (215.9, 168.9)
- moved SC7 19.1 mm to (170.2, 168.9)
Routing:
- net VSS: track 53.0 -> 116.2 mm, vias 7 -> 14
- net Net-(D1-Pad1): track 70.8 -> 32.1 mm
- net Net-(D1-Pad2): track 68.4 -> 34.2 mm
- net VCC: track 26.5 -> 10.8 mm
Other:
- net class Default removed
