File: schematic/Sidepanels_2019/X-/X-.kicad_sch (KiCad schematic)
At the start: 10 parts

Commit message: Push of all changes made for June update
Major change was in the solar cell and creating a new library based on the old one.
Parts:
- D15: value (none) -> D_Photo; footprint (none) -> Diode_SMD:D_0805_2012Metric
- J1: value (none) -> Conn_01x04; footprint (none) -> Connector_Molex:Molex_PicoBlade_53398-0471_1x04-1MP_P1.25mm_Vertical
- J2: value (none) -> Conn_01x02; footprint (none) -> Connector_Molex:Molex_PicoBlade_53398-0271_1x02-1MP_P1.25mm_Vertical
- SC1, SC2, SC3, SC4, SC5, SC6, SC7: value (none) -> Solar_Cell
Changed lines of the file:
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@@
       (effects (font (size 1.27 1.27)) (justify left))
     )
-    (property "Value" "" (id 1) (at 105.6132 100.203 0)
+    (property "Value" "Solar_Cell" (id 1) (at 105.6132 100.203 0)
       (effects (font (size 1.27 1.27)) (justify left))
     )
@@
       (effects (font (size 1.27 1.27)) (justify left))
     )
-    (property "Value" "" (id 1) (at 86.5632 100.203 0)
+    (property "Value" "Solar_Cell" (id 1) (at 86.5632 100.203 0)
       (effects (font (size 1.27 1.27)) (justify left))
     )
@@
       (effects (font (size 1.27 1.27)) hide)
     )
-    (property "Value" "" (id 1) (at 93.1418 90.8558 0))
+    (property "Value" "VCC" (id 1) (at 93.1418 90.8558 0))
     (property "Footprint" "" (id 2) (at 92.71 95.25 0)
       (effects (font (size 1.27 1.27)) hide)
@@
       (effects (font (size 1.27 1.27)) hide)
     )
-    (property "Value" "" (id 1) (at 89.7128 107.2642 0))
+    (property "Value" "VSS" (id 1) (at 89.7128 107.2642 0))
     (property "Footprint" "" (id 2) (at 90.17 102.87 0)
       (effects (font (size 1.27 1.27)) hide)
@@
     (in_bom yes) (on_board yes)
     (property "Reference" "J1" (id 0) (at 93.5228 69.215 0))
-    (property "Value" "" (id 1) (at 93.5228 71.5264 0))
-    (property "Footprint" "" (id 2) (at 91.44 80.01 0)
+    (property "Value" "Conn_01x04" (id 1) (at 93.5228 71.5264 0))
+    (property "Footprint" "Connector_Molex:Molex_PicoBlade_53398-0471_1x04-1MP_P1.25mm_Vertical" (id 2) (at 91.44 80.01 0)
       (effects (font (size 1.27 1.27)) hide)
     )
@@
       (effects (font (size 1.27 1.27)) hide)
     )
-    (property "Value" "" (id 1) (at 102.3112 82.9818 90)
+    (property "Value" "VSS" (id 1) (at 102.3112 82.9818 90)
       (effects (font (size 1.27 1.27)) (justify left))
     )
@@
       (effects (font (size 1.27 1.27)) hide)
     )
-    (property "Value" "" (id 1) (at 102.3112 75.3618 90)
+    (property "Value" "VCC" (id 1) (at 102.3112 75.3618 90)
       (effects (font (size 1.27 1.27)) (justify left))
     )
@@
     (in_bom yes) (on_board yes)
     (property "Reference" "J2" (id 0) (at 94.7928 120.015 0))
-    (property "Value" "" (id 1) (at 94.7928 122.3264 0))
-    (property "Footprint" "" (id 2) (at 92.71 128.27 0)
+    (property "Value" "Conn_01x02" (id 1) (at 94.7928 122.3264 0))
+    (property "Footprint" "Connector_Molex:Molex_PicoBlade_53398-0271_1x02-1MP_P1.25mm_Vertical" (id 2) (at 92.71 128.27 0)
       (effects (font (size 1.27 1.27)) hide)
     )
@@
       (effects (font (size 1.27 1.27)) (justify left))
     )
-    (property "Value" "" (id 1) (at 114.4778 128.143 90)
-      (effects (font (size 1.27 1.27)) (justify left))
-    )
-    (property "Footprint" "" (id 2) (at 110.49 127 0)
+    (property "Value" "D_Photo" (id 1) (at 114.4778 128.143 90)
+      (effects (font (size 1.27 1.27)) (justify left))
+    )
+    (property "Footprint" "Diode_SMD:D_0805_2012Metric" (id 2) (at 110.49 127 0)
       (effects (font (size 1.27 1.27)) hide)
     )
@@
       (effects (font (size 1.27 1.27)) (justify left))
     )
-    (property "Value" "" (id 1) (at 123.3932 100.203 0)
+    (property "Value" "Solar_Cell" (id 1) (at 123.3932 100.203 0)
       (effects (font (size 1.27 1.27)) (justify left))
     )
@@
       (effects (font (size 1.27 1.27)) (justify left))
     )
-    (property "Value" "" (id 1) (at 139.9032 100.203 0)
+    (property "Value" "Solar_Cell" (id 1) (at 139.9032 100.203 0)
       (effects (font (size 1.27 1.27)) (justify left))
     )
@@
       (effects (font (size 1.27 1.27)) (justify left))
     )
-    (property "Value" "" (id 1) (at 157.6832 100.203 0)
+    (property "Value" "Solar_Cell" (id 1) (at 157.6832 100.203 0)
       (effects (font (size 1.27 1.27)) (justify left))
     )
@@
       (effects (font (size 1.27 1.27)) (justify left))
     )
-    (property "Value" "" (id 1) (at 174.1932 100.203 0)
+    (property "Value" "Solar_Cell" (id 1) (at 174.1932 100.203 0)
       (effects (font (size 1.27 1.27)) (justify left))
     )
@@
       (effects (font (size 1.27 1.27)) (justify left))
     )
-    (property "Value" "" (id 1) (at 189.4332 100.203 0)
+    (property "Value" "Solar_Cell" (id 1) (at 189.4332 100.203 0)
       (effects (font (size 1.27 1.27)) (justify left))
     )
@@
     )
     (path "/00000000-0000-0000-0000-00005ca8e593"
-      (reference "SC1") (unit 1) (value "Solar_Cell") (footprint "CySat_Solar:Spectrolab")
+      (reference "SC1") (unit 1) (value "Solar_Cell") (footprint "CySat:Spectrolabs_UTJ")
     )
     (path "/00000000-0000-0000-0000-00005ca8e00b"
-      (reference "SC2") (unit 1) (value "Solar_Cell") (footprint "CySat_Solar:Spectrolab")
+      (reference "SC2") (unit 1) (value "Solar_Cell") (footprint "CySat:Spectrolabs_UTJ")
     )
     (path "/00000000-0000-0000-0000-00005f045ba0"
-      (reference "SC3") (unit 1) (value "Solar_Cell") (footprint "CySat_Solar:Spectrolab")
+      (reference "SC3") (unit 1) (value "Solar_Cell") (footprint "CySat:Spectrolabs_UTJ")
     )
     (path "/00000000-0000-0000-0000-00005f046cfc"
-      (reference "SC4") (unit 1) (value "Solar_Cell") (footprint "CySat_Solar:Spectrolab")
+      (reference "SC4") (unit 1) (value "Solar_Cell") (footprint "CySat:Spectrolabs_UTJ")
     )
     (path "/00000000-0000-0000-0000-00005f04774b"
-      (reference "SC5") (unit 1) (value "Solar_Cell") (footprint "CySat_Solar:Spectrolab")
+      (reference "SC5") (unit 1) (value "Solar_Cell") (footprint "CySat:Spectrolabs_UTJ")
     )
     (path "/00000000-0000-0000-0000-00005f048cbd"
-      (reference "SC6") (unit 1) (value "Solar_Cell") (footprint "CySat_Solar:Spectrolab")
+      (reference "SC6") (unit 1) (value "Solar_Cell") (footprint "CySat:Spectrolabs_UTJ")
     )
     (path "/00000000-0000-0000-0000-00005f049574"
-      (reference "SC7") (unit 1) (value "Solar_Cell") (footprint "CySat_Solar:Spectrolab")
-    )
-  )
+      (reference "SC7") (unit 1) (value "Solar_Cell") (footprint "CySat:Spectrolabs_UTJ")
+    )
+  )
