File: schematic/Sidepanels_2019/Y+/Y+.kicad_pcb (KiCad board)
At the start: 2 copper layers, 327.5 x 83 mm, 42 parts, among them J1 Conn_01x04, J2 Conn_01x02

Commit message: Flipped and/or added TrisolX cells
Parts:
- added D20: D_Schottky, CySat footprints:Toshiba_CUS08F30, B.Cu at (39.5, 83.8)
- added D21: D_Schottky, CySat footprints:Toshiba_CUS08F30, B.Cu at (36.3, 83.8)
- added SC22: Solar_Cell, CySat footprints:TriSelectSolarPanel_Left_Handed, F.Cu at (160.9, 92.9)
- added SC23: Solar_Cell, CySat footprints:TriSelectSolarPanel_Left_Handed, F.Cu at (312.5, 69.4)
Routing:
- net VSS: track 98.3 -> 107.5 mm, vias 24 -> 26
- net VCC: track 43.0 -> 47.0 mm, vias 20 -> 22
Changed lines of the file:
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@@
     (thickness 1.6)
     (drawings 132)
-    (tracks 165)
+    (tracks 177)
     (zones 0)
-    (modules 42)
+    (modules 46)
     (nets 5)
   )
   (page A4)
   (layers
-    (0 F.Cu signal)
+    (0 F.Cu signal hide)
     (31 B.Cu signal hide)
     (32 B.Adhes user)
@@
     (add_net VCC)
     (add_net VSS)
+  )
+  (module "CySat footprints:TriSelectSolarPanel_Left_Handed" (layer F.Cu)
+    (at 312.5131 69.3876 90)
+    (fp_text reference SC23 (at 9.936 0.012 90) (layer F.SilkS)
+      (effects (font (size 1 1) (thickness 0.15)))
+    )
+    (fp_text value Solar_Cell (at -4.796 0.012 90) (layer F.Fab)
+      (effects (font (size 1 1) (thickness 0.15)))
+    )
+    (fp_line (start 13.05 -4.85) (end 13.05 -0.75) (layer F.SilkS) (width 0.12))
+    (fp_line (start 16.15 -4.85) (end 13.05 -4.85) (layer F.SilkS) (width 0.12))
+    (fp_line (start 16.15 -0.75) (end 16.15 -4.85) (layer F.SilkS) (width 0.12))
+    (fp_line (start 11.968 -0.75) (end 16.15 -0.75) (layer F.SilkS) (width 0.12))
+    (fp_line (start -10.25 -5.75) (end -14.75 -0.75) (layer F.SilkS) (width 0.15))
+    (fp_line (start -4.5 -8) (end -10.25 -5.75) (layer F.SilkS) (width 0.15))
+    (fp_line (start 12 -8) (end -4.5 -8) (layer F.SilkS) (width 0.15))
+    (fp_line (start 12 -0.75) (end 12 -8) (layer F.SilkS) (width 0.15))
+    (fp_line (start -14.732 -0.75) (end 11.968 -0.75) (layer F.SilkS) (width 0.15))
+    (pad 1 smd rect (at 3.5 -4.5 90) (size 8.5 3) (layers F.Cu F.Paste F.Mask)
+      (net 2 VCC))
+    (pad 2 smd rect (at 14.6 -2.8 90) (size 3 4) (layers F.Cu F.Paste F.Mask)
+      (net 1 VSS))
+  )
+  (module "CySat footprints:TriSelectSolarPanel_Left_Handed" (layer F.Cu)
+    (at 160.9259 92.9461 90)
+    (fp_text reference SC22 (at 9.936 0.012 90) (layer F.SilkS)
+      (effects (font (size 1 1) (thickness 0.15)))
+    )
+    (fp_text value Solar_Cell (at -4.796 0.012 90) (layer F.Fab)
+      (effects (font (size 1 1) (thickness 0.15)))
+    )
+    (fp_line (start 13.05 -4.85) (end 13.05 -0.75) (layer F.SilkS) (width 0.12))
+    (fp_line (start 16.15 -4.85) (end 13.05 -4.85) (layer F.SilkS) (width 0.12))
+    (fp_line (start 16.15 -0.75) (end 16.15 -4.85) (layer F.SilkS) (width 0.12))
+    (fp_line (start 11.968 -0.75) (end 16.15 -0.75) (layer F.SilkS) (width 0.12))
+    (fp_line (start -10.25 -5.75) (end -14.75 -0.75) (layer F.SilkS) (width 0.15))
+    (fp_line (start -4.5 -8) (end -10.25 -5.75) (layer F.SilkS) (width 0.15))
+    (fp_line (start 12 -8) (end -4.5 -8) (layer F.SilkS) (width 0.15))
+    (fp_line (start 12 -0.75) (end 12 -8) (layer F.SilkS) (width 0.15))
+    (fp_line (start -14.732 -0.75) (end 11.968 -0.75) (layer F.SilkS) (width 0.15))
+    (pad 1 smd rect (at 3.5 -4.5 90) (size 8.5 3) (layers F.Cu F.Paste F.Mask)
+      (net 2 VCC))
+    (pad 2 smd rect (at 14.6 -2.8 90) (size 3 4) (layers F.Cu F.Paste F.Mask)
+      (net 1 VSS))
+  )
+  (module "CySat footprints:Toshiba_CUS08F30" (layer B.Cu)
+    (at 36.3093 83.827 90)
+    (fp_text reference D21 (at 0 -1.65 90) (layer B.SilkS)
+      (effects (font (size 1 1) (thickness 0.15)) (justify mirror))
+    )
+    (fp_text value D_Schottky (at 0 1.5 90) (layer B.Fab)
+      (effects (font (size 1 1) (thickness 0.15)) (justify mirror))
+    )
+    (fp_line (start -1.6 0.5) (end -1.6 -0.5) (layer B.SilkS) (width 0.12))
+    (fp_line (start -0.7 -0.5) (end -0.7 0.5) (layer B.SilkS) (width 0.12))
+    (fp_line (start -1.15 -0.5) (end -0.7 -0.5) (layer B.SilkS) (width 0.12))
+    (fp_line (start -0.7 0.5) (end -1.6 0.5) (layer B.SilkS) (width 0.12))
+    (fp_line (start -1.6 -0.5) (end -1.15 -0.5) (layer B.SilkS) (width 0.12))
+    (fp_line (start 1.6 0.5) (end 1.15 0.5) (layer B.SilkS) (width 0.12))
+    (fp_line (start 1.6 -0.5) (end 1.6 0.5) (layer B.SilkS) (width 0.12))
+    (fp_line (start 0.7 -0.5) (end 1.6 -0.5) (layer B.SilkS) (width 0.12))
+    (fp_line (start 0.7 0.5) (end 0.7 -0.5) (layer B.SilkS) (width 0.12))
+    (fp_line (start 1.15 0.5) (end 0.7 0.5) (layer B.SilkS) (width 0.12))
+    (pad 2 smd rect (at -1.15 0 90) (size 0.9 1) (layers B.Cu B.Paste B.Mask)
+      (net 1 VSS))
+    (pad 1 smd rect (at 1.15 0 90) (size 0.9 1) (layers B.Cu B.Paste B.Mask)
+      (net 2 VCC))
+  )
+  (module "CySat footprints:Toshiba_CUS08F30" (layer B.Cu)
+    (at 39.4716 83.8073 90)
+    (fp_text reference D20 (at 0 -1.65 90) (layer B.SilkS)
+      (effects (font (size 1 1) (thickness 0.15)) (justify mirror))
+    )
+    (fp_text value D_Schottky (at 0 1.5 90) (layer B.Fab)
+      (effects (font (size 1 1) (thickness 0.15)) (justify mirror))
+    )
+    (fp_line (start -1.6 0.5) (end -1.6 -0.5) (layer B.SilkS) (width 0.12))
+    (fp_line (start -0.7 -0.5) (end -0.7 0.5) (layer B.SilkS) (width 0.12))
+    (fp_line (start -1.15 -0.5) (end -0.7 -0.5) (layer B.SilkS) (width 0.12))
+    (fp_line (start -0.7 0.5) (end -1.6 0.5) (layer B.SilkS) (width 0.12))
+    (fp_line (start -1.6 -0.5) (end -1.15 -0.5) (layer B.SilkS) (width 0.12))
+    (fp_line (start 1.6 0.5) (end 1.15 0.5) (layer B.SilkS) (width 0.12))
+    (fp_line (start 1.6 -0.5) (end 1.6 0.5) (layer B.SilkS) (width 0.12))
+    (fp_line (start 0.7 -0.5) (end 1.6 -0.5) (layer B.SilkS) (width 0.12))
+    (fp_line (start 0.7 0.5) (end 0.7 -0.5) (layer B.SilkS) (width 0.12))
+    (fp_line (start 1.15 0.5) (end 0.7 0.5) (layer B.SilkS) (width 0.12))
+    (pad 2 smd rect (at -1.15 0 90) (size 0.9 1) (layers B.Cu B.Paste B.Mask)
+      (net 1 VSS))
+    (pad 1 smd rect (at 1.15 0 90) (size 0.9 1) (layers B.Cu B.Paste B.Mask)
+      (net 2 VCC))
   )
   (module "CySat footprints:Toshiba_CUS08F30" (layer B.Cu)
@@
   (segment (start -6.2812 54.645) (end -2.4542 54.645) (width 0.25) (layer F.Cu) (net 1))
   (segment (start -2.4542 54.645) (end -2.45364 54.64556) (width 0.25) (layer F.Cu) (net 1))
+  (via (at 304.5968 54.7878) (size 0.8) (drill 0.4) (layers F.Cu B.Cu) (net 1))
+  (segment (start 309.7131 54.7876) (end 304.597 54.7876) (width 0.25) (layer F.Cu) (net 1))
+  (segment (start 304.597 54.7876) (end 304.5968 54.7878) (width 0.25) (layer F.Cu) (net 1))
+  (via (at 158.7627 74.5998) (size 0.8) (drill 0.4) (layers F.Cu B.Cu) (net 1))
+  (segment (start 158.1259 78.3461) (end 158.1259 75.2366) (width 0.25) (layer F.Cu) (net 1))
+  (segment (start 158.1259 75.2366) (end 158.7627 74.5998) (width 0.25) (layer F.Cu) (net 1))
   (via (at 40.9956 63.4111) (size 0.8) (drill 0.4) (layers F.Cu B.Cu) (net 2))
   (segment (start 39.05 63.45) (end 40.9567 63.45) (width 0.25) (layer B.Cu) (net 2))
@@
   (segment (start 30.45 88.225) (end 31.94924 86.72576) (width 0.25) (layer B.Cu) (net 2))
   (segment (start 31.94924 86.72576) (end 32.50692 86.72576) (width 0.25) (layer B.Cu) (net 2))
+  (via (at 41.6179 82.677) (size 0.8) (drill 0.4) (layers F.Cu B.Cu) (net 2))
+  (segment (start 39.4716 82.6573) (end 41.5982 82.6573) (width 0.25) (layer B.Cu) (net 2))
+  (segment (start 41.5982 82.6573) (end 41.6179 82.677) (width 0.25) (layer B.Cu) (net 2))
+  (via (at 34.4297 82.7278) (size 0.8) (drill 0.4) (layers F.Cu B.Cu) (net 2))
+  (segment (start 36.3093 82.677) (end 34.4805 82.677) (width 0.25) (layer B.Cu) (net 2))
+  (segment (start 34.4805 82.677) (end 34.4297 82.7278) (width 0.25) (layer B.Cu) (net 2))
   (segment (start 30.45 78.275) (end 32.30644 78.275) (width 0.25) (layer B.Cu) (net 3))
   (segment (start 32.30644 78.275) (end 32.36976 78.21168) (width 0.25) (layer B.Cu) (net 3))

Commit message: Fixed Trisol Cells
Parts:
- removed D20, D21: D_Schottky, CySat footprints:Toshiba_CUS08F30
- removed SC22, SC23: Solar_Cell, CySat footprints:TriSelectSolarPanel_Left_Handed
Routing:
- net VSS: track 107.5 -> 102.3 mm, vias 26 -> 25
- net VCC: track 47.0 -> 43.0 mm, vias 22 -> 20
Changed lines of the file:
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@@
     (thickness 1.6)
     (drawings 132)
-    (tracks 177)
+    (tracks 168)
     (zones 0)
-    (modules 46)
+    (modules 42)
     (nets 5)
   )
   (page A4)
   (layers
-    (0 F.Cu signal hide)
-    (31 B.Cu signal hide)
+    (0 F.Cu signal)
+    (31 B.Cu signal)
     (32 B.Adhes user)
     (33 F.Adhes user)
@@
     (add_net VCC)
     (add_net VSS)
-  )
-  (module "CySat footprints:TriSelectSolarPanel_Left_Handed" (layer F.Cu)
-    (at 312.5131 69.3876 90)
-    (fp_text reference SC23 (at 9.936 0.012 90) (layer F.SilkS)
-      (effects (font (size 1 1) (thickness 0.15)))
-    )
-    (fp_text value Solar_Cell (at -4.796 0.012 90) (layer F.Fab)
-      (effects (font (size 1 1) (thickness 0.15)))
-    )
-    (fp_line (start 13.05 -4.85) (end 13.05 -0.75) (layer F.SilkS) (width 0.12))
-    (fp_line (start 16.15 -4.85) (end 13.05 -4.85) (layer F.SilkS) (width 0.12))
-    (fp_line (start 16.15 -0.75) (end 16.15 -4.85) (layer F.SilkS) (width 0.12))
-    (fp_line (start 11.968 -0.75) (end 16.15 -0.75) (layer F.SilkS) (width 0.12))
-    (fp_line (start -10.25 -5.75) (end -14.75 -0.75) (layer F.SilkS) (width 0.15))
-    (fp_line (start -4.5 -8) (end -10.25 -5.75) (layer F.SilkS) (width 0.15))
-    (fp_line (start 12 -8) (end -4.5 -8) (layer F.SilkS) (width 0.15))
-    (fp_line (start 12 -0.75) (end 12 -8) (layer F.SilkS) (width 0.15))
-    (fp_line (start -14.732 -0.75) (end 11.968 -0.75) (layer F.SilkS) (width 0.15))
-    (pad 1 smd rect (at 3.5 -4.5 90) (size 8.5 3) (layers F.Cu F.Paste F.Mask)
-      (net 2 VCC))
-    (pad 2 smd rect (at 14.6 -2.8 90) (size 3 4) (layers F.Cu F.Paste F.Mask)
-      (net 1 VSS))
-  )
-  (module "CySat footprints:TriSelectSolarPanel_Left_Handed" (layer F.Cu)
-    (at 160.9259 92.9461 90)
-    (fp_text reference SC22 (at 9.936 0.012 90) (layer F.SilkS)
-      (effects (font (size 1 1) (thickness 0.15)))
-    )
-    (fp_text value Solar_Cell (at -4.796 0.012 90) (layer F.Fab)
-      (effects (font (size 1 1) (thickness 0.15)))
-    )
-    (fp_line (start 13.05 -4.85) (end 13.05 -0.75) (layer F.SilkS) (width 0.12))
-    (fp_line (start 16.15 -4.85) (end 13.05 -4.85) (layer F.SilkS) (width 0.12))
-    (fp_line (start 16.15 -0.75) (end 16.15 -4.85) (layer F.SilkS) (width 0.12))
-    (fp_line (start 11.968 -0.75) (end 16.15 -0.75) (layer F.SilkS) (width 0.12))
-    (fp_line (start -10.25 -5.75) (end -14.75 -0.75) (layer F.SilkS) (width 0.15))
-    (fp_line (start -4.5 -8) (end -10.25 -5.75) (layer F.SilkS) (width 0.15))
-    (fp_line (start 12 -8) (end -4.5 -8) (layer F.SilkS) (width 0.15))
-    (fp_line (start 12 -0.75) (end 12 -8) (layer F.SilkS) (width 0.15))
-    (fp_line (start -14.732 -0.75) (end 11.968 -0.75) (layer F.SilkS) (width 0.15))
-    (pad 1 smd rect (at 3.5 -4.5 90) (size 8.5 3) (layers F.Cu F.Paste F.Mask)
-      (net 2 VCC))
-    (pad 2 smd rect (at 14.6 -2.8 90) (size 3 4) (layers F.Cu F.Paste F.Mask)
-      (net 1 VSS))
-  )
-  (module "CySat footprints:Toshiba_CUS08F30" (layer B.Cu)
-    (at 36.3093 83.827 90)
-    (fp_text reference D21 (at 0 -1.65 90) (layer B.SilkS)
-      (effects (font (size 1 1) (thickness 0.15)) (justify mirror))
-    )
-    (fp_text value D_Schottky (at 0 1.5 90) (layer B.Fab)
-      (effects (font (size 1 1) (thickness 0.15)) (justify mirror))
-    )
-    (fp_line (start -1.6 0.5) (end -1.6 -0.5) (layer B.SilkS) (width 0.12))
-    (fp_line (start -0.7 -0.5) (end -0.7 0.5) (layer B.SilkS) (width 0.12))
-    (fp_line (start -1.15 -0.5) (end -0.7 -0.5) (layer B.SilkS) (width 0.12))
-    (fp_line (start -0.7 0.5) (end -1.6 0.5) (layer B.SilkS) (width 0.12))
-    (fp_line (start -1.6 -0.5) (end -1.15 -0.5) (layer B.SilkS) (width 0.12))
-    (fp_line (start 1.6 0.5) (end 1.15 0.5) (layer B.SilkS) (width 0.12))
-    (fp_line (start 1.6 -0.5) (end 1.6 0.5) (layer B.SilkS) (width 0.12))
-    (fp_line (start 0.7 -0.5) (end 1.6 -0.5) (layer B.SilkS) (width 0.12))
-    (fp_line (start 0.7 0.5) (end 0.7 -0.5) (layer B.SilkS) (width 0.12))
-    (fp_line (start 1.15 0.5) (end 0.7 0.5) (layer B.SilkS) (width 0.12))
-    (pad 2 smd rect (at -1.15 0 90) (size 0.9 1) (layers B.Cu B.Paste B.Mask)
-      (net 1 VSS))
-    (pad 1 smd rect (at 1.15 0 90) (size 0.9 1) (layers B.Cu B.Paste B.Mask)
-      (net 2 VCC))
-  )
-  (module "CySat footprints:Toshiba_CUS08F30" (layer B.Cu)
-    (at 39.4716 83.8073 90)
-    (fp_text reference D20 (at 0 -1.65 90) (layer B.SilkS)
-      (effects (font (size 1 1) (thickness 0.15)) (justify mirror))
-    )
-    (fp_text value D_Schottky (at 0 1.5 90) (layer B.Fab)
-      (effects (font (size 1 1) (thickness 0.15)) (justify mirror))
-    )
-    (fp_line (start -1.6 0.5) (end -1.6 -0.5) (layer B.SilkS) (width 0.12))
-    (fp_line (start -0.7 -0.5) (end -0.7 0.5) (layer B.SilkS) (width 0.12))
-    (fp_line (start -1.15 -0.5) (end -0.7 -0.5) (layer B.SilkS) (width 0.12))
-    (fp_line (start -0.7 0.5) (end -1.6 0.5) (layer B.SilkS) (width 0.12))
-    (fp_line (start -1.6 -0.5) (end -1.15 -0.5) (layer B.SilkS) (width 0.12))
-    (fp_line (start 1.6 0.5) (end 1.15 0.5) (layer B.SilkS) (width 0.12))
-    (fp_line (start 1.6 -0.5) (end 1.6 0.5) (layer B.SilkS) (width 0.12))
-    (fp_line (start 0.7 -0.5) (end 1.6 -0.5) (layer B.SilkS) (width 0.12))
-    (fp_line (start 0.7 0.5) (end 0.7 -0.5) (layer B.SilkS) (width 0.12))
-    (fp_line (start 1.15 0.5) (end 0.7 0.5) (layer B.SilkS) (width 0.12))
-    (pad 2 smd rect (at -1.15 0 90) (size 0.9 1) (layers B.Cu B.Paste B.Mask)
-      (net 1 VSS))
-    (pad 1 smd rect (at 1.15 0 90) (size 0.9 1) (layers B.Cu B.Paste B.Mask)
-      (net 2 VCC))
   )
   (module "CySat footprints:Toshiba_CUS08F30" (layer B.Cu)
@@
   (segment (start -6.2812 54.645) (end -2.4542 54.645) (width 0.25) (layer F.Cu) (net 1))
   (segment (start -2.4542 54.645) (end -2.45364 54.64556) (width 0.25) (layer F.Cu) (net 1))
-  (via (at 304.5968 54.7878) (size 0.8) (drill 0.4) (layers F.Cu B.Cu) (net 1))
-  (segment (start 309.7131 54.7876) (end 304.597 54.7876) (width 0.25) (layer F.Cu) (net 1))
-  (segment (start 304.597 54.7876) (end 304.5968 54.7878) (width 0.25) (layer F.Cu) (net 1))
   (via (at 158.7627 74.5998) (size 0.8) (drill 0.4) (layers F.Cu B.Cu) (net 1))
   (segment (start 158.1259 78.3461) (end 158.1259 75.2366) (width 0.25) (layer F.Cu) (net 1))
@@
   (segment (start 30.45 88.225) (end 31.94924 86.72576) (width 0.25) (layer B.Cu) (net 2))
   (segment (start 31.94924 86.72576) (end 32.50692 86.72576) (width 0.25) (layer B.Cu) (net 2))
-  (via (at 41.6179 82.677) (size 0.8) (drill 0.4) (layers F.Cu B.Cu) (net 2))
-  (segment (start 39.4716 82.6573) (end 41.5982 82.6573) (width 0.25) (layer B.Cu) (net 2))
-  (segment (start 41.5982 82.6573) (end 41.6179 82.677) (width 0.25) (layer B.Cu) (net 2))
-  (via (at 34.4297 82.7278) (size 0.8) (drill 0.4) (layers F.Cu B.Cu) (net 2))
-  (segment (start 36.3093 82.677) (end 34.4805 82.677) (width 0.25) (layer B.Cu) (net 2))
-  (segment (start 34.4805 82.677) (end 34.4297 82.7278) (width 0.25) (layer B.Cu) (net 2))
   (segment (start 30.45 78.275) (end 32.30644 78.275) (width 0.25) (layer B.Cu) (net 3))
   (segment (start 32.30644 78.275) (end 32.36976 78.21168) (width 0.25) (layer B.Cu) (net 3))

Commit message: Update to Y+
Parts:
- removed D10, D11, D12, D13, D14, D15, D16, D17, D18, D2, D3, D4, D5, D6, D7, D8, D9: D_Schottky, CySat footprints:Toshiba_CUS08F30
- removed D19: D_Photo, CySat footprints:Sun_Sensor
- removed SC10, SC11, SC12, SC13, SC14, SC15, SC16, SC17, SC18, SC5, SC6, SC7, SC8, SC9: Solar_Cell, CySat footprints:TriSelectSolarPanel
- removed SC19, SC20, SC21: Solar_Cell, CySat footprints:Spectrolab
- D1: value D_Schottky -> D_Photo; footprint CySat footprints:Toshiba_CUS08F30 -> Diode_SMD:D_0805_2012Metric; moved to F.Cu
- SC1, SC2, SC3, SC4: footprint CySat footprints:TriSelectSolarPanel -> CySat_Solar:Spectrolab
- moved D1 289.8 mm to (278.8, 251.5), turned to 270 degrees
- moved SC3 228.9 mm to (302.9, 227.3)
- moved SC1 211.5 mm to (266.7, 228.0), turned to 0 degrees
- moved SC2 196.9 mm to (234.3, 225.4), turned to 180 degrees
- moved J1 195.8 mm to (166.4, 229.8)
- moved J2 195.8 mm to (166.4, 218.6)
- moved SC4 174.2 mm to (163.2, 224.2), turned to 180 degrees
Connections:
- D1 pad 1: VCC -> Net-(D1-Pad1)
- D1 pad 2: VSS -> Net-(D1-Pad2)
- J2 pad 1: Net-(D19-Pad2) -> Net-(D1-Pad2)
- J2 pad 2: Net-(D19-Pad1) -> Net-(D1-Pad1)
Routing:
- net Net-(D1-Pad2): track 0.00 -> 124.9 mm, vias 0 -> 1
- net Net-(D1-Pad1): track 0.00 -> 124.8 mm, vias 0 -> 1
- net VSS: track 102.3 -> 30.0 mm, vias 25 -> 4
- net Net-(D19-Pad2): track 49.9 -> 0.00 mm, vias 1 -> 0
- net Net-(D19-Pad1): track 46.2 -> 0.00 mm, vias 1 -> 0
- net VCC: track 43.0 -> 32.1 mm, vias 20 -> 1
Other:
- outline, holes or cut-outs redrawn
- board text added: "CySat Panel Y+"
- board text added: "CySat-1 Make to Innovate Iowa State University"
- board text added: "I figure if a farmer’s daughter from Iowa can become an astronaut, you can be just about anything you want to be. - Peggy Whitson"

Commit message: Added cutout to y+
Generated Gerber files
Other:
- outline, holes or cut-outs redrawn

Commit message: update to y+
Other:
- rule pad_to_mask_clearance: 0.051 -> 0
Changed lines of the file:
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@@
     (pad_size 1.524 1.524)
     (pad_drill 0.762)
-    (pad_to_mask_clearance 0.051)
-    (solder_mask_min_width 0.25)
+    (pad_to_mask_clearance 0)
     (aux_axis_origin 0 0)
     (visible_elements 7FFFFFFF)
@@
       (outputformat 1)
       (mirror false)
-      (drillshape 1)
+      (drillshape 0)
       (scaleselection 1)
-      (outputdirectory ""))
+      (outputdirectory "gerber/"))
   )
   (net 0 "")
@@
     (pad 4 smd roundrect (at 1.875 1.25 90) (size 0.8 1.3) (layers B.Cu B.Paste B.Mask) (roundrect_rratio 0.25)
       (net 2 VCC))
-    (pad MP smd roundrect (at -4.425 -1.5 90) (size 2.1 3) (layers B.Cu B.Paste B.Mask) (roundrect_rratio 0.119048))
-    (pad MP smd roundrect (at 4.425 -1.5 90) (size 2.1 3) (layers B.Cu B.Paste B.Mask) (roundrect_rratio 0.119048))
+    (pad MP smd roundrect (at -4.425 -1.5 90) (size 2.1 3) (layers B.Cu B.Paste B.Mask) (roundrect_rratio 0.119047619047619))
+    (pad MP smd roundrect (at 4.425 -1.5 90) (size 2.1 3) (layers B.Cu B.Paste B.Mask) (roundrect_rratio 0.119047619047619))
     (model ${KISYS3DMOD}/Connector_Molex.3dshapes/Molex_PicoBlade_53398-0471_1x04-1MP_P1.25mm_Vertical.wrl
       (at (xyz 0 0 0))
@@
       (effects (font (size 1 1) (thickness 0.15)) (justify mirror))
     )
-    (pad MP smd roundrect (at 3.175 -1.5 90) (size 2.1 3) (layers B.Cu B.Paste B.Mask) (roundrect_rratio 0.119048))
-    (pad MP smd roundrect (at -3.175 -1.5 90) (size 2.1 3) (layers B.Cu B.Paste B.Mask) (roundrect_rratio 0.119048))
+    (pad MP smd roundrect (at 3.175 -1.5 90) (size 2.1 3) (layers B.Cu B.Paste B.Mask) (roundrect_rratio 0.119047619047619))
+    (pad MP smd roundrect (at -3.175 -1.5 90) (size 2.1 3) (layers B.Cu B.Paste B.Mask) (roundrect_rratio 0.119047619047619))
     (pad 2 smd roundrect (at 0.625 1.25 90) (size 0.8 1.3) (layers B.Cu B.Paste B.Mask) (roundrect_rratio 0.25)
       (net 3 "Net-(D1-Pad1)"))

Commit message: Push of all changes made for June update
Major change was in the solar cell and creating a new library based on the old one.
Parts:
- SC1, SC2, SC3, SC4: footprint CySat_Solar:Spectrolab -> CySat:Spectrolabs_UTJ
- moved D1 103.3 mm to (180.6, 219.4)
- moved SC1 30.3 mm to (245.6, 206.2)
- moved SC4 22.2 mm to (161.2, 246.3)
- moved SC3 21.9 mm to (324.8, 228.0)
- moved SC2 21.8 mm to (233.2, 247.2)
- moved J1 0.06 mm to (166.3, 229.8)
Routing:
- net VSS: track 30.0 -> 199.4 mm, vias 4 -> 2
- net Net-(D1-Pad1): track 124.8 -> 13.2 mm
- net Net-(D1-Pad2): track 124.9 -> 14.0 mm
- net VCC: track 32.1 -> 5.55 mm
Other:
- net class Default removed
